File: kicad/24-24-converter/24-24-converter.kicad_pcb (KiCad board)
At the start: 4 copper layers, 143.5 x 76 mm, 81 parts, among them J1 Conn_01x02, J2 Conn_01x02, J3 Enable, M1 CSD18540Q5B, M1_1 CSD18540Q5B, M2 CSD18540Q5B, M2_1 CSD18540Q5B, M3 GENERIC_MOSFET_N, M3_1 GENERIC_MOSFET_N, M4 GENERIC_MOSFET_N, U1 LM5176PWPR

Commit message: fixedenable connector issue
Parts:
- moved Cf1 0.71 mm to (142.0, 114.0)
Connections:
- J3 pad 1: Enable -> /EN
- J3 pad 2: /EN -> GND
Routing:
- net /HDRV1: track 70.0 -> 66.3 mm
- net GND: track 31.3 -> 32.9 mm, vias 638 -> 639
- net /EN: track 39.8 -> 39.5 mm, vias 2 -> 1
Changed lines of the file:
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@@
 			(layers "*.Cu" "*.Mask")
 			(remove_unused_layers no)
-			(net "Enable")
+			(net "/EN")
 			(pinfunction "Pin_1_1")
 			(pintype "passive")
@@
 			(layers "*.Cu" "*.Mask")
 			(remove_unused_layers no)
-			(net "/EN")
+			(net "GND")
 			(pinfunction "Pin_2_2")
 			(pintype "passive")
@@
 	(footprint "Capacitor_SMD:C_0805_2012Metric_Pad1.18x1.45mm_HandSolder"
 		(layer "B.Cu")
-		(at 141.5 114.5 -90)
+		(at 142 114 -90)
 		(descr "Capacitor SMD 0805 (2012 Metric), square (rectangular) end terminal, IPC-7351 nominal with elongated pad for handsoldering. (Body size source: IPC-SM-782 page 76, https://www.pcb-3d.com/wordpress/wp-content/uploads/ipc-sm-782a_amendment_1_and_2.pdf, https://docs.google.com/spreadsheets/d/1BsfQQcO9C6DZCsRaXUlFlo91Tg2WpOkGARC1WS5S8t0/edit?usp=sharing)")
 		(tags "capacitor handsolder")
@@
 	)
 	(via
-		(at 140.2875 115.5375)
+		(at 140.5 115)
 		(size 0.6)
 		(drill 0.3)
@@
 	)
 	(via
+		(at 150 126.5)
+		(size 0.6)
+		(drill 0.3)
+		(layers "F.Cu" "B.Cu")
+		(net "GND")
+	)
+	(via
 		(at 73.5 84.5)
 		(size 0.6)
@@
 	)
 	(segment
+		(start 140.5375 115.0375)
+		(end 140.5 115)
+		(width 0.2)
+		(layer "B.Cu")
+		(net "GND")
+	)
+	(segment
 		(start 137.3375 98.4125)
 		(end 137 98.75)
@@
 	)
 	(segment
-		(start 141.5 115.5375)
-		(end 140.2875 115.5375)
-		(width 0.2)
-		(layer "B.Cu")
-		(net "GND")
-	)
-	(segment
 		(start 137.3375 111)
 		(end 136 109.6625)
@@
 	)
 	(segment
+		(start 142 115.0375)
+		(end 140.5375 115.0375)
+		(width 0.2)
+		(layer "B.Cu")
+		(net "GND")
+	)
+	(segment
+		(start 148.75 126.5)
+		(end 150 126.5)
+		(width 0.2)
+		(layer "B.Cu")
+		(net "GND")
+	)
+	(segment
 		(start 152.25 107.25)
 		(end 153.25 108.25)
@@
 	)
 	(segment
-		(start 129.6 112.6)
-		(end 126 109)
-		(width 0.2)
-		(layer "F.Cu")
-		(net "/HDRV1")
-	)
-	(segment
 		(start 120.015 73.801)
 		(end 120.63 74.416)
@@
 	)
 	(segment
-		(start 146.9 112.6)
-		(end 129.6 112.6)
+		(start 120.015 73.43)
+		(end 120.015 73.801)
 		(width 0.2)
 		(layer "F.Cu")
@@
 	)
 	(segment
-		(start 120.015 73.43)
-		(end 120.015 73.801)
+		(start 146.9 112.6)
+		(end 149 110.5)
 		(width 0.2)
 		(layer "F.Cu")
@@
 	)
 	(segment
-		(start 120.63 74.416)
-		(end 126 74.416)
+		(start 135 111.75)
+		(end 135.85 112.6)
 		(width 0.2)
 		(layer "F.Cu")
@@
 	)
 	(segment
-		(start 149 110.5)
+		(start 135.85 112.6)
 		(end 146.9 112.6)
 		(width 0.2)
@@
 		(net "/HDRV1")
 	)
+	(segment
+		(start 120.63 74.416)
+		(end 126 74.416)
+		(width 0.2)
+		(layer "F.Cu")
+		(net "/HDRV1")
+	)
 	(via
-		(at 126 109)
+		(at 135 111.75)
 		(size 0.6)
 		(drill 0.3)
@@
 	)
 	(segment
-		(start 126 75)
-		(end 126 109)
+		(start 135 111.75)
+		(end 126 102.75)
+		(width 0.2)
+		(layer "In2.Cu")
+		(net "/HDRV1")
+	)
+	(segment
+		(start 126 102.75)
+		(end 126 75)
 		(width 0.2)
 		(layer "In2.Cu")
@@
 		(net "/EN")
 	)
-	(via
-		(at 142.5 112)
-		(size 0.6)
-		(drill 0.3)
-		(layers "F.Cu" "B.Cu")
-		(net "/EN")
-	)
 	(segment
 		(start 141.5 100)
@@
 	)
 	(segment
-		(start 142.125 101.125)
-		(end 142.125 100.625)
+		(start 142.4475 111.5525)
+		(end 141.800001 110.905)
 		(width 0.2)
 		(layer "B.Cu")
@@
 	)
 	(segment
-		(start 142.5 112)
-		(end 142.5 111.604999)
+		(start 142.4475 111.5525)
+		(end 147.75 116.855)
 		(width 0.2)
 		(layer "B.Cu")
@@
 	)
 	(segment
-		(start 142.5 111.604999)
-		(end 141.800001 110.905)
+		(start 147.75 116.855)
+		(end 147.75 126.5)
 		(width 0.2)
 		(layer "B.Cu")
@@
 	(segment
 		(start 142.125 101.125)
-		(end 139.1625 98.1625)
+		(end 142.125 100.625)
 		(width 0.2)
 		(layer "B.Cu")
@@
 	)
 	(segment
-		(start 139.1625 98.1625)
-		(end 139.1625 96.75)
+		(start 142.5 111.604999)
+		(end 142.4475 111.5525)
 		(width 0.2)
 		(layer "B.Cu")
@@
 	)
 	(segment
-		(start 142.5 112)
-		(end 148.75 118.25)
+		(start 142.125 101.125)
+		(end 139.1625 98.1625)
 		(width 0.2)
-		(layer "In2.Cu")
+		(layer "B.Cu")
 		(net "/EN")
 	)
 	(segment
-		(start 148.75 118.25)
-		(end 148.75 126.5)
+		(start 139.1625 98.1625)
+		(end 139.1625 96.75)
 		(width 0.2)
-		(layer "In2.Cu")
+		(layer "B.Cu")
 		(net "/EN")
 	)
@@
 	(segment
 		(start 141.5 112)
-		(end 141.5 113.4625)
+		(end 140.800001 111.300001)
 		(width 0.2)
 		(layer "B.Cu")
@@
 	)
 	(segment
-		(start 141.5 112)
-		(end 140.800001 111.300001)
+		(start 152.5 98.75)
+		(end 152.75 98.75)
 		(width 0.2)
 		(layer "B.Cu")
@@
 	)
 	(segment
-		(start 152.5 98.75)
-		(end 152.75 98.75)
+		(start 141.5 112.4625)
+		(end 142 112.9625)
 		(width 0.2)
 		(layer "B.Cu")
@@
 	)
 	(segment
+		(start 141.5 112)
+		(end 141.5 112.4625)
+		(width 0.2)
+		(layer "B.Cu")
+		(net "Net-(U1-VIN)")
+	)
+	(segment
 		(start 140.900001 110.254999)
 		(end 141.800001 110.254999)
@@
 		(net "Net-(U1-VINSNS)")
 	)
-	(segment
-		(start 140.473001 112)
-		(end 140.473001 112.223001)
-		(width 0.2)
-		(layer "B.Cu")
-		(net "Net-(U1-VINSNS)")
-	)

Commit message: Routing Attempt #4
Parts:
- removed Ruvb1: CRCW040215K0FKED, Resistor_SMD:R_0603_1608Metric_Pad0.98x0.95mm_HandSolder
- moved Ruvt1 18.2 mm to (144.2, 114.2), turned to 90 degrees
- moved Rvisns1 18.1 mm to (139.0, 114.8), turned to 90 degrees
- moved D2 0.56 mm to (156.5, 103.8)
- moved Cboot2 0.25 mm to (151.5, 105.2)
Routing:
- net VIN: track 32.2 -> 65.5 mm
- net /EN: track 39.5 -> 18.1 mm, vias 1 -> 0
- net Net-(U1-VINSNS): track 19.1 -> 5.90 mm, vias 2 -> 0
- net GND: track 32.9 -> 30.1 mm
- net Net-(D2-K): track 6.91 -> 7.83 mm

Commit message: fixed enable issue
Routing:
- net VOUT: track 50.1 -> 54.7 mm, vias 88 -> 90
- net /LDRV2: track 33.3 -> 31.8 mm, vias 4 -> 2
Changed lines of the file:
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@@
 		(net "VOUT")
 	)
+	(segment
+		(start 154.75 95.25)
+		(end 157 95.25)
+		(width 0.2)
+		(layer "F.Cu")
+		(net "VOUT")
+	)
 	(via
 		(at 164.25 77.75)
@@
 	)
 	(via
+		(at 154.75 95.25)
+		(size 0.6)
+		(drill 0.3)
+		(layers "F.Cu" "B.Cu")
+		(net "VOUT")
+	)
+	(via
 		(at 198 79)
 		(size 0.6)
@@
 	)
 	(via
+		(at 157 95.25)
+		(size 0.6)
+		(drill 0.3)
+		(layers "F.Cu" "B.Cu")
+		(net "VOUT")
+	)
+	(via
 		(at 202.5 68.5)
 		(size 0.6)
@@
 	)
 	(segment
+		(start 156.75 88.25)
+		(end 157.25 88.75)
+		(width 0.2)
+		(layer "B.Cu")
+		(net "VOUT")
+	)
+	(segment
 		(start 140.900001 103.755)
 		(end 140.670001 103.525)
@@
 	)
 	(segment
+		(start 157.25 95)
+		(end 157 95.25)
+		(width 0.2)
+		(layer "B.Cu")
+		(net "VOUT")
+	)
+	(segment
+		(start 157.25 88.75)
+		(end 157.25 95)
+		(width 0.2)
+		(layer "B.Cu")
+		(net "VOUT")
+	)
+	(segment
 		(start 141.800001 103.755)
 		(end 140.900001 103.755)
@@
 	)
 	(segment
-		(start 141.5 103.5)
-		(end 140.5 103.5)
+		(start 141.796471 103.525)
+		(end 150.071471 95.25)
+		(width 0.2)
+		(layer "In2.Cu")
+		(net "VOUT")
+	)
+	(segment
+		(start 140.5 103.525)
+		(end 141.796471 103.525)
 		(width 0.2)
 		(layer "In2.Cu")
@@
 	)
 	(segment
-		(start 156.75 88.25)
-		(end 141.5 103.5)
+		(start 150.071471 95.25)
+		(end 154.75 95.25)
 		(width 0.2)
 		(layer "In2.Cu")
@@
 	)
 	(segment
-		(start 156.25 98.5875)
-		(end 156.25 94.598529)
+		(start 156.25 94.598529)
+		(end 156.25 98.5875)
 		(width 0.2)
 		(layer "B.Cu")
@@
 	)
 	(via
-		(at 154.5 89.651473)
-		(size 0.6)
-		(drill 0.3)
-		(layers "F.Cu" "B.Cu")
-		(net "/LDRV2")
-	)
-	(via
 		(at 154.305 80.805)
 		(size 0.6)
@@
 		(net "/LDRV2")
 	)
-	(via
-		(at 157 94.75)
-		(size 0.6)
-		(drill 0.3)
-		(layers "F.Cu" "B.Cu")
-		(net "/LDRV2")
-	)
-	(segment
-		(start 156.75 94.5)
-		(end 156.75 91.401471)
-		(width 0.2)
-		(layer "B.Cu")
-		(net "/LDRV2")
-	)
-	(segment
-		(start 155.000002 89.651473)
-		(end 154.5 89.651473)
-		(width 0.2)
-		(layer "B.Cu")
-		(net "/LDRV2")
-	)
-	(segment
-		(start 156.75 91.401471)
-		(end 155.000002 89.651473)
-		(width 0.2)
-		(layer "B.Cu")
-		(net "/LDRV2")
-	)
 	(segment
 		(start 148.895001 106.354999)
@@
 	)
 	(segment
-		(start 157 94.75)
-		(end 156.75 94.5)
-		(width 0.2)
-		(layer "B.Cu")
-		(net "/LDRV2")
-	)
-	(segment
-		(start 156.75 95)
-		(end 156.75 98.5)
+		(start 154.5 94)
+		(end 154.5 81)
 		(width 0.2)
 		(layer "In2.Cu")
@@
 	)
 	(segment
-		(start 156.75 98.5)
+		(start 155.5 99.75)
 		(end 149.25 106)
 		(width 0.2)
@@
 	)
 	(segment
-		(start 154.5 89.651473)
-		(end 154.5 81)
+		(start 155.5 95)
+		(end 155.5 99.75)
 		(width 0.2)
 		(layer "In2.Cu")
@@
 	)
 	(segment
-		(start 157 94.75)
-		(end 156.75 95)
+		(start 155.5 95)
+		(end 154.5 94)
 		(width 0.2)
 		(layer "In2.Cu")

Commit message: Fixed chip footprint
Parts:
- added Ruvb1: CRCW040215K0FKED, Resistor_SMD:R_0603_1608Metric_Pad0.98x0.95mm_HandSolder, B.Cu at (146.5, 114.5)
- moved U1 0.18 mm to (144.8, 106.5)
Routing:
- net Net-(U1-RT_SYNC): track 3.36 -> 4.00 mm
- net GND: track 30.1 -> 30.2 mm, vias 639 -> 643

Commit message: Thermal Relief on Connectors
Parts:
- moved J1 0.94 mm to (75.8, 70.0)
Routing:
- net VOUT: vias 90 -> 110
- net GND: vias 643 -> 657

Commit message: Added Alignment Holes and created Gerbers
Parts:
- added H5: Alignment Hole, 24V_Converter:Alignment Hole, F.Cu at (183.4, 59.6)
- added H6: Alignment Hole, 24V_Converter:Alignment Hole, F.Cu at (75.8, 103.0)
- added H7: Alignment Hole, 24V_Converter:Alignment Hole, F.Cu at (166.2, 120.2)
