File: kicad/24-24-converter/24-24-converter.kicad_sch (KiCad schematic)
At the start: 78 parts, among them J1 Conn_01x02, J2 Conn_01x02, M1 CSD18540Q5B, M1_1 CSD18540Q5B, M2 CSD18540Q5B, M2_1 CSD18540Q5B, M3 GENERIC_MOSFET_N, M3_1 GENERIC_MOSFET_N, M4 GENERIC_MOSFET_N, U1 LM5176PWPR

Commit message: import project files, remove template project
Other:
- note removed: "24V Converter"
- company: (none) -> Mars Rover Club Electrical Team
- title: (none) -> ${MRC_TITLE}

Commit message: added filled zones
Other:
- moved on the sheet: Cout1, Cout_1, Cout_2, D3, J2, R2

Commit message: Routing Attempt #3
Connections:
- net SW2: now also M4.9 (Drain)
- net VOUT: now also M3.9 (Drain), M3_1.9 (Drain)
Changed lines of the file:
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@@
 	)
 	(symbol
+		(lib_name "root_0_M3_TI WEBENCH_1")
 		(lib_id "TI WEBENCH:root_0_M3_TI WEBENCH")
 		(at 132.08 73.66 0)
@@
 		(pin "8"
 		)
+		(pin "9"
+		)
 		(instances
 			(project "24-24-converter"
@@
 		(pin "8"
 		)
+		(pin "9"
+		)
 		(instances
 			(project "24-24-converter"
@@
 	)
 	(symbol
+		(lib_name "root_0_M3_TI WEBENCH_2")
 		(lib_id "TI WEBENCH:root_0_M3_TI WEBENCH")
 		(at 132.08 48.26 0)
@@
 		(pin "8"
 		)
+		(pin "9"
+		)
 		(instances

Commit message: Routing Attempt #5
Parts:
- removed Cbulk1: 50SVPF10M, 24V_Converter:Cbulk_CAP_B6-SVPK_PAN, symbol Device:C_Polarized_US
- removed Cin_5: 50SVPF39M, 24V_Converter:Cin_50SVPF39M, symbol Device:C_Polarized_US
- added C13: 50SVPF39M, 24V_Converter:Cin_50SVPF39M, symbol Device:C_Polarized_US
- added C7: 50SVPF10M, 24V_Converter:Cbulk_CAP_B6-SVPK_PAN, symbol Device:C_Polarized_US
- added J3: Enable, Connector_AMASS:AMASS_XT30U-M_1x02_P5.0mm_Vertical, symbol Connector_Generic:Conn_01x02
- renumbered Cbulk_1 to C1, Coutx_2 to C10, Coutx_3 to C11, Coutx_4 to C12, Cin1 to C14, Cin_1 to C15, Cin_2 to C16, Cin_3 to C17, Cin_4 to C18, Coutx2 to C19, Cbulk_2 to C2, Coutx3_1 to C20, Coutx3_2 to C21, Coutx3_3 to C22, Coutx3_4 to C23, Coutx3 to C24, Coutx2_1 to C25, Coutx2_2 to C26, Coutx2_3 to C27, Coutx2_4 to C28, Cout1 to C29, Cbulk_3 to C3, Cout_1 to C30, Cout_2 to C31, Ccomp1 to C32, Ccomp_1 to C33, Ccomp2 to C34, Cbulk_4 to C4, Cbulk_5 to C5, Cbulk_6 to C6, Coutx1 to C8, Coutx_1 to C9
Connections:
- net EN: now also J3.2 (Pin_2)
- net GND: now also C13.2, C7.2
- net VIN: now also C13.1, C7.1
- new net Enable: J3.1 (Pin_1)

Commit message: fixedenable connector issue
Parts:
- J3: footprint Connector_AMASS:AMASS_XT30U-M_1x02_P5.0mm_Vertical -> Connector_PinHeader_1.00mm:PinHeader_1x02_P1.00mm_Vertical
Connections:
- net Enable is gone; now on net EN: J3.1 (Pin_1)
- net EN: no longer J3.2 (Pin_2)
- net GND: now also J3.2 (Pin_2)
Other:
- moved on the sheet: J3
Changed lines of the file:
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@@
 	)
 	(junction
-		(at 36.83 29.21)
-		(diameter 0)
-		(color 0 0 0 0)
-	)
-	(junction
 		(at 34.29 91.44)
 		(diameter 0)
@@
 	)
 	(junction
+		(at 36.83 29.21)
+		(diameter 0)
+		(color 0 0 0 0)
+	)
+	(junction
 		(at 49.53 91.44)
 		(diameter 0)
@@
 	(wire
 		(pts
-			(xy 48.26 22.86) (xy 48.26 29.21)
-		)
-		(stroke
-			(width 0)
-			(type default)
-		)
-	)
-	(wire
-		(pts
 			(xy 142.24 31.75) (xy 142.24 34.29)
 		)
@@
 	(wire
 		(pts
-			(xy 36.83 29.21) (xy 48.26 29.21)
-		)
-		(stroke
-			(width 0)
-			(type default)
-		)
-	)
-	(wire
-		(pts
 			(xy 72.39 162.56) (xy 77.47 162.56)
 		)
@@
 	(wire
 		(pts
+			(xy 36.83 29.21) (xy 46.99 29.21)
+		)
+		(stroke
+			(width 0)
+			(type default)
+		)
+	)
+	(wire
+		(pts
 			(xy 151.13 63.5) (xy 151.13 58.42)
 		)
@@
 	(wire
 		(pts
+			(xy 36.83 29.21) (xy 36.83 31.75)
+		)
+		(stroke
+			(width 0)
+			(type default)
+		)
+	)
+	(wire
+		(pts
+			(xy 46.99 31.75) (xy 46.99 35.56)
+		)
+		(stroke
+			(width 0)
+			(type default)
+		)
+	)
+	(wire
+		(pts
 			(xy 29.21 62.23) (xy 29.21 66.04)
 		)
@@
 	(wire
 		(pts
-			(xy 36.83 29.21) (xy 36.83 31.75)
-		)
-		(stroke
-			(width 0)
-			(type default)
-		)
-	)
-	(wire
-		(pts
 			(xy 95.25 53.34) (xy 95.25 58.42)
 		)
@@
 	(symbol
 		(lib_id "Connector_Generic:Conn_01x02")
-		(at 53.34 20.32 0)
+		(at 52.07 29.21 0)
 		(unit 1)
 		(body_style 1)
@@
 		(fields_autoplaced yes)
 		(property "Reference" "J3"
-			(at 55.88 20.3199 0)
+			(at 54.61 29.2099 0)
 			(show_name no)
 			(do_not_autoplace no)
@@
 		)
 		(property "Value" "Enable"
-			(at 55.88 22.8599 0)
+			(at 54.61 31.7499 0)
 			(show_name no)
 			(do_not_autoplace no)
@@
 			)
 		)
-		(property "Footprint" "Connector_AMASS:AMASS_XT30U-M_1x02_P5.0mm_Vertical"
-			(at 53.34 20.32 0)
+		(property "Footprint" "Connector_PinHeader_1.00mm:PinHeader_1x02_P1.00mm_Vertical"
+			(at 52.07 29.21 0)
 			(hide yes)
 			(show_name no)
@@
 		)
 		(property "Datasheet" ""
-			(at 53.34 20.32 0)
+			(at 52.07 29.21 0)
 			(hide yes)
 			(show_name no)
@@
 		)
 		(property "Description" "Generic connector, single row, 01x02, script generated (kicad-library-utils/schlib/autogen/connector/)"
-			(at 53.34 20.32 0)
+			(at 52.07 29.21 0)
 			(hide yes)
 			(show_name no)
@@
 	)
 	(symbol
-		(lib_id "power:+28V")
-		(at 48.26 20.32 0)
-		(unit 1)
-		(body_style 1)
-		(exclude_from_sim no)
-		(in_bom yes)
-		(on_board yes)
-		(in_pos_files yes)
-		(dnp no)
-		(property "Reference" "#PWR035"
-			(at 48.26 24.13 0)
-			(hide yes)
-			(show_name no)
-			(do_not_autoplace no)
-			(effects
-				(font
-					(size 1.27 1.27)
-				)
-			)
-		)
-		(property "Value" "Enable"
-			(at 52.324 17.78 0)
-			(show_name no)
-			(do_not_autoplace no)
-			(effects
-				(font
-					(size 1.27 1.27)
-				)
-			)
-		)
-		(property "Footprint" ""
-			(at 54.61 19.05 0)
-			(hide yes)
-			(show_name no)
-			(do_not_autoplace no)
-			(effects
-				(font
-					(size 1.27 1.27)
-				)
-			)
-		)
-		(property "Datasheet" ""
-			(at 54.61 19.05 0)
-			(hide yes)
-			(show_name no)
-			(do_not_autoplace no)
-			(effects
-				(font
-					(size 1.27 1.27)
-				)
-			)
-		)
-		(property "Description" "Power symbol creates a global label with name \"+28V\""
-			(at 48.26 20.32 0)
-			(hide yes)
-			(show_name no)
-			(do_not_autoplace no)
-			(effects
-				(font
-					(size 1.27 1.27)
-				)
-			)
-		)
-		(pin "1"
-		)
-		(instances
-			(project "24-24-converter"
-				(path "/9e6f5c11-8bef-4e05-9856-b93512fc7502"
-					(reference "#PWR035")
-					(unit 1)
-				)
-			)
-		)
-	)
-	(symbol
 		(lib_name "root_0_M3_TI WEBENCH_2")
 		(lib_id "TI WEBENCH:root_0_M3_TI WEBENCH")
@@
 					(unit 1)
 				)
+			)
+		)
+	)
+	(symbol
+		(lib_id "power:GND")
+		(at 46.99 35.56 0)
+		(unit 1)
+		(body_style 1)
+		(exclude_from_sim no)
+		(in_bom yes)
+		(on_board yes)
+		(in_pos_files yes)
+		(dnp no)
+		(property "Reference" "#PWR035"
+			(at 46.99 41.91 0)
+			(hide yes)
+			(show_name no)
+			(do_not_autoplace no)
+			(effects
+				(font
+					(size 1.27 1.27)
+				)
+			)
+		)
+		(property "Value" "GND"
+			(at 51.308 36.576 0)
+			(show_name no)
+			(do_not_autoplace no)
+			(effects
+				(font
+					(size 1.27 1.27)
+				)
+			)
+		)
+		(property "Footprint" ""
+			(at 46.99 35.56 0)
+			(hide yes)
+			(show_name no)
+			(do_not_autoplace no)
+			(effects
+				(font
+					(size 1.27 1.27)
+				)
+			)
+		)
+		(property "Datasheet" ""
+			(at 46.99 35.56 0)
+			(hide yes)
+			(show_name no)
+			(do_not_autoplace no)
+			(effects
+				(font
+					(size 1.27 1.27)
+				)
+			)
+		)
+		(property "Description" "Power symbol creates a global label with name \"GND\" , ground"
+			(at 46.99 35.56 0)
+			(hide yes)
+			(show_name no)
+			(do_not_autoplace no)
+			(effects
+				(font
+					(size 1.27 1.27)
+				)
+			)
+		)
+		(pin "1"
+		)
+		(instances
+			(project "24-24-converter"
+				(path "/9e6f5c11-8bef-4e05-9856-b93512fc7502"
+					(reference "#PWR035")
+					(unit 1)
+				)

Commit message: Added Alignment Holes and created Gerbers
Parts:
- added H5, H6, H7: Alignment Hole, 24V_Converter:Alignment Hole, symbol Mechanical:MountingHole
Changed lines of the file:
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@@
 	)
 	(symbol
+		(lib_id "Mechanical:MountingHole")
+		(at 170.18 220.98 0)
+		(unit 1)
+		(body_style 1)
+		(exclude_from_sim no)
+		(in_bom no)
+		(on_board yes)
+		(in_pos_files yes)
+		(dnp no)
+		(fields_autoplaced yes)
+		(property "Reference" "H7"
+			(at 172.72 219.7099 0)
+			(show_name no)
+			(do_not_autoplace no)
+			(effects
+				(font
+					(size 1.27 1.27)
+				)
+				(justify left)
+			)
+		)
+		(property "Value" "Alignment Hole"
+			(at 172.72 222.2499 0)
+			(show_name no)
+			(do_not_autoplace no)
+			(effects
+				(font
+					(size 1.27 1.27)
+				)
+				(justify left)
+			)
+		)
+		(property "Footprint" "24V_Converter:Alignment Hole"
+			(at 170.18 220.98 0)
+			(hide yes)
+			(show_name no)
+			(do_not_autoplace no)
+			(effects
+				(font
+					(size 1.27 1.27)
+				)
+			)
+		)
+		(property "Datasheet" ""
+			(at 170.18 220.98 0)
+			(hide yes)
+			(show_name no)
+			(do_not_autoplace no)
+			(effects
+				(font
+					(size 1.27 1.27)
+				)
+			)
+		)
+		(property "Description" "Mounting Hole without connection"
+			(at 170.18 220.98 0)
+			(hide yes)
+			(show_name no)
+			(do_not_autoplace no)
+			(effects
+				(font
+					(size 1.27 1.27)
+				)
+			)
+		)
+		(instances
+			(project "24-24-converter"
+				(path "/9e6f5c11-8bef-4e05-9856-b93512fc7502"
+					(reference "H7")
+					(unit 1)
+				)
+			)
+		)
+	)
+	(symbol
 		(lib_id "TI WEBENCH:root_0_M2_TI WEBENCH")
 		(at 91.44 73.66 0)
@@
 	)
 	(symbol
+		(lib_id "Mechanical:MountingHole")
+		(at 170.18 207.01 0)
+		(unit 1)
+		(body_style 1)
+		(exclude_from_sim no)
+		(in_bom no)
+		(on_board yes)
+		(in_pos_files yes)
+		(dnp no)
+		(fields_autoplaced yes)
+		(property "Reference" "H5"
+			(at 172.72 205.7399 0)
+			(show_name no)
+			(do_not_autoplace no)
+			(effects
+				(font
+					(size 1.27 1.27)
+				)
+				(justify left)
+			)
+		)
+		(property "Value" "Alignment Hole"
+			(at 172.72 208.2799 0)
+			(show_name no)
+			(do_not_autoplace no)
+			(effects
+				(font
+					(size 1.27 1.27)
+				)
+				(justify left)
+			)
+		)
+		(property "Footprint" "24V_Converter:Alignment Hole"
+			(at 170.18 207.01 0)
+			(hide yes)
+			(show_name no)
+			(do_not_autoplace no)
+			(effects
+				(font
+					(size 1.27 1.27)
+				)
+			)
+		)
+		(property "Datasheet" ""
+			(at 170.18 207.01 0)
+			(hide yes)
+			(show_name no)
+			(do_not_autoplace no)
+			(effects
+				(font
+					(size 1.27 1.27)
+				)
+			)
+		)
+		(property "Description" "Mounting Hole without connection"
+			(at 170.18 207.01 0)
+			(hide yes)
+			(show_name no)
+			(do_not_autoplace no)
+			(effects
+				(font
+					(size 1.27 1.27)
+				)
+			)
+		)
+		(instances
+			(project "24-24-converter"
+				(path "/9e6f5c11-8bef-4e05-9856-b93512fc7502"
+					(reference "H5")
+					(unit 1)
+				)
+			)
+		)
+	)
+	(symbol
 		(lib_id "Device:C_Polarized_US")
 		(at 78.74 58.42 0)
@@
 					(unit 1)
 				)
+			)
+		)
+	)
+	(symbol
+		(lib_id "Mechanical:MountingHole")
+		(at 170.18 213.36 0)
+		(unit 1)
+		(body_style 1)
+		(exclude_from_sim no)
+		(in_bom no)
+		(on_board yes)
+		(in_pos_files yes)
+		(dnp no)
+		(fields_autoplaced yes)
+		(property "Reference" "H6"
+			(at 172.72 212.0899 0)
+			(show_name no)
+			(do_not_autoplace no)
+			(effects
+				(font
+					(size 1.27 1.27)
+				)
+				(justify left)
+			)
+		)
+		(property "Value" "Alignment Hole"
+			(at 172.72 214.6299 0)
+			(show_name no)
+			(do_not_autoplace no)
+			(effects
+				(font
+					(size 1.27 1.27)
+				)
+				(justify left)
+			)
+		)
+		(property "Footprint" "24V_Converter:Alignment Hole"
+			(at 170.18 213.36 0)
+			(hide yes)
+			(show_name no)
+			(do_not_autoplace no)
+			(effects
+				(font
+					(size 1.27 1.27)
+				)
+			)
+		)
+		(property "Datasheet" ""
+			(at 170.18 213.36 0)
+			(hide yes)
+			(show_name no)
+			(do_not_autoplace no)
+			(effects
+				(font
+					(size 1.27 1.27)
+				)
+			)
+		)
+		(property "Description" "Mounting Hole without connection"
+			(at 170.18 213.36 0)
+			(hide yes)
+			(show_name no)
+			(do_not_autoplace no)
+			(effects
+				(font
+					(size 1.27 1.27)
+				)
+			)
+		)
+		(instances
+			(project "24-24-converter"
+				(path "/9e6f5c11-8bef-4e05-9856-b93512fc7502"
+					(reference "H6")
+					(unit 1)
+				)
